File: Hardware/jf-ecu32/jf-ecu32.kicad_sch (KiCad schematic)
At the start: 72 parts, among them J1 GAZ, J10 k, J11 RPM, J12 S.PORT, J13 PPM/PWM, J14 PUMP1, J15 PUMP1, J16 PPM/PWM, J17 PUMP2, J18 PUMP2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

Commit message: PCB
Parts:
- removed D17: BZV55C3V3, Diode_SMD:D_MiniMELF, symbol Diode:BZV55C3V3
- added C?: 0.1µF, Capacitor_SMD:CP_Elec_5x3, symbol Device:C
- added C?: 22µF, Capacitor_SMD:C_0603_1608Metric, symbol Device:C
- added C?: 0.1µF, Capacitor_SMD:C_0603_1608Metric, symbol Device:C
- added D?: SMF5V0A, Diode_SMD:D_SMF, symbol Diode:SMF5V0A
- added U?: BMP280, Package_LGA:Bosch_LGA-8_2x2.5mm_P0.65mm_ClockwisePinNumbering, symbol Sensor_Pressure:BMP280
Connections:
- net +3.3V: now also D?.1 (A1)
- net CLK: now also U1.30 (IO18), U?.4 (SCK); no longer U1.29 (IO5)
- net CS: now also U1.29 (IO5); no longer U1.37 (IO23)
- net GLOW_CURRENT: now also U1.5 (SENSOR_VN); no longer U1.23 (IO15)
- net GND: now also C?.2, C?.2, C?.2, D?.2 (A2), U?.1 (GND), U?.7 (GND)
- net MISO: now also U?.5 (SDO)
- net VBAT_ADC: now also U1.4 (SENSOR_VP); no longer U1.26 (IO4)
- net V_CPU: now also C?.1, C?.1, C?.1, U?.6 (VDDIO), U?.8 (VDD)
- new net MOSI: U1.37 (IO23), U?.3 (SDI)
Other:
- moved on the sheet: C7, R5
