File: Hardware/jf-ecu32/jf-ecu32.kicad_sch (KiCad schematic)
At the start: 69 parts, among them J1 GAZ, J10 k, J11 RPM, J12 S.PORT, J13 PPM/PWM, J14 PUMP1, J15 PUMP1, J16 PPM/PWM, J17 PUMP2, J18 PUMP2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

Commit message: PCB
Parts:
- added C10, C11, C5, C6: 0.1µF, Capacitor_SMD:C_0603_1608Metric, symbol Device:C
- added GND, TCK, TDO, TMS: Conn_01x01_Male, Connector_PinHeader_1.00mm:PinHeader_1x01_P1.00mm_Vertical, symbol Connector:Conn_01x01_Male
- added TDI: Conn_01x01_Male, symbol Connector:Conn_01x01_Male
Connections:
- net +3.3V: now also C11.1, C5.1, C6.1
- net GND: now also C11.2, C5.2, C6.2, GND.1 (Pin_1)
- net PWM_KEROSTART_3.3: now also TMS.1 (Pin_1)
- net PWM_KERO_3.3: now also TDI.1 (Pin_1)
- net at J10.1 (Pin_1), U3.2 (T-): now also C10.2
- net at J10.2 (Pin_2), U3.3 (T+): now also C10.1
- net TCK: now reaches U1.16 (IO13)
- net TCK: now also TCK.1 (Pin_1)
- net TDO: now reaches U1.23 (IO15)
- net TDO: now also TDO.1 (Pin_1)

Commit message: PCB
Parts:
- removed C4: 22µF, Capacitor_SMD:CP_Elec_5x3, symbol Device:C
- removed D17: SMF5V0A, Diode_SMD:D_SMF, symbol Diode:SMF5V0A
- added D1: SMF5V0A, Diode_SMD:D_SMF, symbol Diode:SMF5V0A
- added U6: AMS1117-5.0, Package_TO_SOT_SMD:SOT-223-3_TabPin2, symbol Regulator_Linear:AMS1117-5.0
- C3: value 0.1µF -> 22µF
- C8: footprint Capacitor_SMD:C_0603_1608Metric -> Capacitor_SMD:CP_Elec_5x3
- TDI1: renamed from TDI; footprint (none) -> Connector_PinHeader_1.00mm:PinHeader_1x01_P1.00mm_Vertical
- renumbered GND to GND1, TCK to TCK1, TDO to TDO1, TMS to TMS1
Connections:
- net +3.3V: no longer C5.1, C8.1, U5.1 (VCC)
- net +BATT: now also U6.3 (VI)
- net GND: now also D1.2 (A2), U6.1 (GND)
- net VDC: no longer U4.3 (VI)
- new net +5V: C5.1, C8.1, D1.1 (A1), U4.3 (VI), U5.1 (VCC), U6.2 (VO)
Other:
- moved on the sheet: C3, C9, D3, Q4, R9

Commit message: PCB
Parts:
- added Q7: AO3401A, Package_TO_SOT_SMD:SOT-23, symbol Transistor_FET:AO3401A
- J19: footprint Connector_PinHeader_2.54mm:PinHeader_1x03_P2.54mm_Vertical -> Connector_PinHeader_2.54mm:PinHeader_1x04_P2.54mm_Vertical; symbol Connector_Generic:Conn_01x03 -> Connector_Generic:Conn_01x04
Connections:
- net +3.3V: now also J19.1 (Pin_1); no longer J11.2 (Pin_2), R14.2
- net +5V: now also J11.2 (Pin_2)
- net +BATT: now also Q7.2 (S)
- net GND: now also J19.4 (Pin_4); no longer J19.3 (Pin_3)
- net at U1.35 (TXD0/IO1): now also J19.2 (Pin_2); no longer J19.1 (Pin_1)
- net at U1.34 (RXD0/IO3): now also J19.3 (Pin_3); no longer J19.2 (Pin_2)
- net at D3.2 (A), J9.1 (Pin_1), Q4.2 (D): now also Q7.3 (D)
- new net V_CPU: R14.2

Commit message: PCB
Parts:
- removed D11, D12, D14, D16, D4, D5, D6, D8: D_Schottky, Diode_SMD:D_SMA, symbol Device:D_Schottky
- added R15, R16: 10K, Resistor_SMD:R_0603_1608Metric, symbol Device:R
Connections:
- net V_CPU is gone; now on net +3.3V: R14.2
- net GND: now also R15.2, R16.1
- net PWM_KERO_3.3: now also R16.2
- net at U1.24 (IO2): now also R15.1
- net BRAKE: now reaches U1.26 (IO4)
- net BRAKE: now also Q7.1 (G)
Other:
- moved on the sheet: R14

Commit message: PCB
Parts:
- added D?: D_Schottky, Diode_SMD:D_SMA, symbol Device:D_Schottky
- added R? (x2): 10k, Resistor_SMD:R_0603_1608Metric, symbol Device:R
- added R?: 50k, Resistor_SMD:R_0603_1608Metric, symbol Device:R
Connections:
- net +5V: now also R?.1
- net +BATT: now also D?.1 (K), R?.1
- net GND: now also R?.2
- new net D2: D?.2 (A), R?.1, R?.2, R?.2

Commit message: PCB V2
Parts:
- removed D?: D_Schottky, Diode_SMD:D_SMA, symbol Device:D_Schottky
- removed R? (x2): 10k, Resistor_SMD:R_0603_1608Metric, symbol Device:R
- removed R?: 50k, Resistor_SMD:R_0603_1608Metric, symbol Device:R
- added BOOT0, GND2: Conn_01x01_Male, Connector_PinHeader_2.00mm:PinHeader_1x01_P2.00mm_Vertical, symbol Connector:Conn_01x01_Male
- GND1, TCK1, TDI1, TDO1, TMS1: footprint Connector_PinHeader_1.00mm:PinHeader_1x01_P1.00mm_Vertical -> Connector_PinHeader_2.00mm:PinHeader_1x01_P2.00mm_Vertical
Connections:
- net GND: now also GND2.1 (Pin_1)
- net at BOOT1.1, R13.2, U1.25 (IO0): now also BOOT0.1 (Pin_1)
Other:
- moved on the sheet: BOOT1

Commit message: PCB V3
Parts:
- added C4: 0.1µF, Capacitor_SMD:C_0603_1608Metric, symbol Device:C
- added R17, R20: 20K, Resistor_SMD:R_0603_1608Metric, symbol Device:R
- added R18: 100, Resistor_SMD:R_0603_1608Metric, symbol Device:R
- added R19: 7K, Resistor_SMD:R_0603_1608Metric, symbol Device:R
- added R21: 510K, Resistor_SMD:R_0603_1608Metric, symbol Device:R
- added R22: 500, Resistor_SMD:R_0603_1608Metric, symbol Device:R
- added U7: OPA340NA, Package_TO_SOT_SMD:SOT-23-5, symbol Amplifier_Operational:OPA340NA
- added U8: LM4040DBZ-2.5, Package_TO_SOT_SMD:SOT-23, symbol Reference_Voltage:LM4040DBZ-2.5
Connections:
- net +5V: now also R22.1, U7.5 (V+)
- net GND: now also R18.1, U7.2 (V-), U8.2 (A)
- net RPM: now also C4.1; no longer U1.33 (IO21)
- new net: R18.2, R19.1
- new net: C4.2, R17.2, U7.4 (-)
- new net: R20.2, R21.1, U7.3 (+)
- new net +2V5: R17.1, R19.2, R20.1, R22.2, U8.1 (K)
- new net RPM-2: R21.2, U1.33 (IO21), U7.1

Commit message: RPM problem
Parts:
- added C12: 0.1µF, Capacitor_SMD:C_0603_1608Metric, symbol Device:C
- R18: value 100 -> 20K
- R19: value 7K -> 20K
- R21: value 510K -> 20K
Connections:
- net +2V5: now also C12.1; no longer R19.2
- net GND: now also R19.1, C12.2; no longer R18.1
- net RPM-2: now also R18.1, R19.2; no longer R21.2, U7.1
- net at R18.2: now also R21.2, U7.1; no longer R19.1
Other:
- moved on the sheet: R20
