File: Hardware/jf-ecu32/jf-ecu32.kicad_pcb (KiCad board)
At the start: 2 copper layers, 27 parts, among them J1 GAZ, J10 k, J11 RPM, J12 S.PORT, J2 AUX, J3 PPM/PWM, J4 STARTER, J5 GLOW, J6 VANNE KEROSTART, J7 VANNE KERO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

Commit message: update
Connections:
- U1 pad 10: unconnected-(U1-Pad10) -> PPM_GAZ
- U1 pad 20: PPM_PWM_PUMP2_3.3 -> unconnected-(U1-Pad20)
- U1 pad 21: PPM_PWM_PUMP1_3.3 -> unconnected-(U1-Pad21)
- U1 pad 22: PWM_KERO_3.3 -> unconnected-(U1-Pad22)
- U1 pad 23: PWM_KEROSTART_3.3 -> unconnected-(U1-Pad23)
- U1 pad 24: PWM_GLOW_3.3 -> unconnected-(U1-Pad24)
- U1 pad 25: PPM_STARTER_3.3 -> PWM_KERO_3.3
- U1 pad 27: RX2 -> PWM_KEROSTART_3.3
- U1 pad 33: unconnected-(U1-Pad33) -> RPM
- U1 pad 36: unconnected-(U1-Pad36) -> AUX
- U1 pad 5: PPM_GAZ -> PPM_PWM_PUMP1_3.3
- U1 pad 6: AUX -> PPM_PWM_PUMP2_3.3
- U1 pad 7: RPM -> PWM_GLOW_3.3
- U1 pad 8: unconnected-(U1-Pad8) -> PPM_STARTER_3.3

Commit message: PCB update
Parts:
- added BT1: Battery_Cell, Battery:Battery_Panasonic_CR2032-VS1N_Vertical_CircularHoles, F.Cu at (50.4, 147.1)
- added D1: D_Schottky, Diode_SMD:D_SMC, F.Cu at (57.1, 151.1)
- added D10: D_Schottky, Diode_SMD:D_SMC, B.Cu at (30.5, 173.4)
- added D11: D_Schottky, Diode_SMD:D_SMC, F.Cu at (56.6, 193.5)
- added D12: D_Schottky, Diode_SMD:D_SMC, F.Cu at (68.6, 159.4)
- added D13: D_Schottky, Diode_SMD:D_SMC, B.Cu at (30.5, 185.4)
- added D14: D_Schottky, Diode_SMD:D_SMC, B.Cu at (46.4, 183.7)
- added D15: D_Schottky, Diode_SMD:D_SMC, B.Cu at (30.7, 191.1)
- added D16: D_Schottky, Diode_SMD:D_SMC, B.Cu at (50.8, 183.7)
- added D2: D_Schottky, Diode_SMD:D_SMC, F.Cu at (44.5, 151.1)
- added D3: D_Schottky, Diode_SMD:D_SMC, B.Cu at (30.5, 179.7)
- added D4: D_Schottky, Diode_SMD:D_SMC, B.Cu at (41.9, 183.7)
- added D5: D_Schottky, Diode_SMD:D_SMC, F.Cu at (80.5, 159.5)
- added D6: D_Schottky, Diode_SMD:D_SMC, F.Cu at (20.1, 157.6)
- added D7: D_Schottky, Diode_SMD:D_SMC, B.Cu at (30.5, 165.7)
- added D8: D_Schottky, Diode_SMD:D_SMC, F.Cu at (74.3, 159.4)
- added D9: D_Schottky, Diode_SMD:D_SMC, B.Cu at (30.5, 169.5)
- added J13: PPM/PWM, Connector_PinHeader_2.54mm:PinHeader_1x03_P2.54mm_Vertical, F.Cu at (52.1, 175.9)
- added J14: PUMP1, Connector_AMASS:AMASS_XT30U-F_1x02_P5.0mm_Vertical, F.Cu at (22.8, 185.4)
- added J15: PUMP1, Connector_PinHeader_2.54mm:PinHeader_1x03_P2.54mm_Vertical, F.Cu at (45.7, 191.2)
- added J16: PPM/PWM, Connector_PinHeader_2.54mm:PinHeader_1x03_P2.54mm_Vertical, F.Cu at (54.6, 175.9)
- added J17: PUMP2, Connector_AMASS:AMASS_XT30U-F_1x02_P5.0mm_Vertical, F.Cu at (22.8, 191.1)
- added J18: PUMP2, Connector_PinHeader_2.54mm:PinHeader_1x03_P2.54mm_Vertical, F.Cu at (48.3, 191.1)
- added Q5: QM6006D, Package_TO_SOT_SMD:TO-252-2, F.Cu at (32.4, 185.7)
- added Q6: QM6006D, Package_TO_SOT_SMD:TO-252-2, F.Cu at (32.4, 192.0)
- added R10: R, Resistor_SMD:R_0603_1608Metric, F.Cu at (38.7, 165.7)
- added R11: R, Resistor_SMD:R_0603_1608Metric, F.Cu at (64.1, 154.9)
- added R12: R, Resistor_SMD:R_0603_1608Metric, F.Cu at (39.4, 158.8)
- added R7: R, Resistor_SMD:R_0603_1608Metric, F.Cu at (38.7, 185.4)
- added R8: R, Resistor_SMD:R_0603_1608Metric, F.Cu at (39.0, 191.6)
- added R9: R, Resistor_SMD:R_0603_1608Metric, F.Cu at (38.1, 179.2)
- R1, R2: value R -> R020
- U1: footprint Espressif:ESP32-DevKitC -> RF_Module:ESP32-WROOM-32
- U2, U3: moved to B.Cu
- moved J4 151.6 mm to (43.2, 191.2)
- moved Q4 138.9 mm to (32.4, 179.1), turned to 180 degrees
- moved U4 133.4 mm to (33.0, 148.0)
- moved J3 132.2 mm to (49.5, 175.9), turned to 180 degrees
- moved Q3 130.4 mm to (32.4, 158.8), turned to 180 degrees
- moved U3 125.8 mm to (71.8, 189.2), turned to -90 degrees
- moved J10 119.8 mm to (41.9, 144.1), turned to -90 degrees
- moved J2 119.3 mm to (72.4, 150.5), turned to 180 degrees
- moved Q1 116.4 mm to (32.4, 165.7), turned to 180 degrees
- moved J1 114.3 mm to (74.9, 150.5), turned to 180 degrees
- moved U5 114.2 mm to (52.1, 161.3)
- moved Q2 113.1 mm to (32.4, 172.3), turned to 180 degrees
- moved J12 92.2 mm to (69.8, 150.5), turned to 180 degrees
- moved U1 90.6 mm to (71.8, 177.8), turned to 180 degrees
- moved J9 89.7 mm to (22.8, 179.7), turned to 180 degrees
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Connections:
- J3 pad 1: PPM_STARTER -> Net-(J3-Pad1)
- J3 pad 2: Net-(J3-Pad2) -> PPM_PWM_STARTER
- J5 pad 1: +BATT -> Net-(D10-Pad2)
- J5 pad 2: Net-(J5-Pad2) -> +BATT
- J8 pad 1: +BATT -> GND
- J8 pad 2: GND -> +BATT
- J9 pad 1: +BATT -> Net-(D3-Pad2)
- J9 pad 2: Net-(J9-Pad2) -> +BATT
- Q2 pad 2: Net-(J5-Pad2) -> Net-(D10-Pad2)
- Q4 pad 1: Net-(J3-Pad2) -> Net-(J3-Pad1)
- Q4 pad 2: Net-(J9-Pad2) -> Net-(D3-Pad2)
- U1 pad 1: +3.3V -> VBAT_ADC
- U5 pad 10: PWM_KERO -> PPM_PWM_STARTER
- U5 pad 2: PPM_STARTER -> PWM_KERO
- U5 pad 3: PPM_STARTER_3.3 -> PWM_KERO_3.3
- U5 pad 9: PWM_KERO_3.3 -> PPM_STARTER_3.3
Routing:
- net +BATT: track 0.00 -> 95.1 mm
- net GND: track 0.00 -> 40.1 mm
- net Net-(J16-Pad1): track 0.00 -> 33.4 mm
- net Net-(D16-Pad1): track 0.00 -> 32.2 mm
- net Net-(D4-Pad1): track 0.00 -> 30.7 mm, vias 0 -> 1
- net Net-(J13-Pad1): track 0.00 -> 26.3 mm
- net Net-(D14-Pad1): track 0.00 -> 26.0 mm
- net Net-(J3-Pad1): track 0.00 -> 17.1 mm
- net Net-(D7-Pad2): track 0.00 -> 14.5 mm
- net Net-(D9-Pad2): track 0.00 -> 13.2 mm
- net Net-(D10-Pad2): track 0.00 -> 12.3 mm
- net Net-(D15-Pad2): track 0.00 -> 11.9 mm
- net Net-(D3-Pad2): track 0.00 -> 11.7 mm
- net Net-(D13-Pad2): track 0.00 -> 11.5 mm
- net PPM_PWM_PUMP2: track 0.00 -> 10.9 mm
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
Commit message: PCB
Parts:
- added C1: C, Capacitor_SMD:C_0603_1608Metric, F.Cu at (40.6, 132.1)
- added C2: C, Capacitor_SMD:C_0603_1608Metric, F.Cu at (44.6, 132.1)
- added C3: 0.1µF, Capacitor_SMD:CP_Elec_5x3, F.Cu at (61.6, 148.0)
- added C4: 22µF, Capacitor_SMD:CP_Elec_5x3, F.Cu at (44.7, 125.9)
- D1, D10, D11, D12, D13, D14, D15, D16, D2, D3, D4, D5, D6, D7, D8, D9: footprint Diode_SMD:D_SMC -> Diode_SMD:D_SMB
- U2, U5: footprint Package_SO:SOP-16_3.9x9.9mm_P1.27mm -> Package_SO:SOP-16_4.4x10.4mm_P1.27mm
- moved J10 58.8 mm to (70.5, 195.6), turned to 90 degrees
- moved U4 36.9 mm to (69.9, 148.6)
- moved D2 15.5 mm to (29.8, 146.1)
- moved BT1 13.7 mm to (58.0, 135.7)
- moved D12 13.4 mm to (81.9, 158.4)
- moved J12 12.1 mm to (81.9, 151.1)
- moved R11 11.4 mm to (52.7, 154.3), turned to 90 degrees
- moved D5 7.52 mm to (73.0, 158.4)
- moved J2 7.02 mm to (79.4, 151.1)
- moved D1 5.25 mm to (54.4, 146.7)
- moved D8 3.34 mm to (77.5, 158.4)
- moved J1 2.01 mm to (76.8, 151.1)
Routing:
- net +3.3V: track 0.00 -> 30.1 mm
- net PPM_GAZ_5V: track 0.00 -> 29.6 mm
- net AUX_5V: track 0.00 -> 28.8 mm
- net PPM_GAZ: track 0.00 -> 19.1 mm, vias 0 -> 1
- net VDC: track 0.00 -> 12.7 mm
- net TX2: track 0.00 -> 5.08 mm
- net PWM_GLOW: track 0.00 -> 3.01 mm
- added copper zone on B.Cu, net GND
- added copper zone on F.Cu, net GND
Other:
- board outline added: 73 x 55.4 mm

Commit message: pcb
Parts:
- added D17: BZV55C3V3, Diode_SMD:D_MiniMELF, F.Cu at (62.6, 160.5)
- D1, D10, D11, D12, D13, D14, D15, D16, D2, D3, D4, D5, D7, D8, D9: footprint Diode_SMD:D_SMB -> Diode_SMD:D_SMA
- D6: footprint Diode_SMD:D_SMB -> Diode_SMD:D_SMA; moved to B.Cu
- Q1, Q3: value QM6006D -> AO3400A; footprint Package_TO_SOT_SMD:TO-252-2 -> Package_TO_SOT_SMD:SOT-23
- U5: moved to B.Cu
- moved J10 60.1 mm to (27.9, 153.2)
- moved U3 48.6 mm to (37.1, 155.2), turned to 0 degrees
- moved D11 44.9 mm to (30.6, 156.9), turned to 0 degrees
- moved C2 35.5 mm to (37.8, 166.9), turned to 90 degrees
- moved C4 29.2 mm to (44.7, 155.1), turned to -90 degrees
- moved C1 26.9 mm to (53.6, 155.7)
- moved R11 23.4 mm to (38.4, 172.8)
- moved D2 15.0 mm to (29.7, 161.0)
- moved R3 13.5 mm to (20.8, 161.3)
- moved R4 13.5 mm to (23.8, 161.3)
- moved R12 11.1 mm to (29.8, 164.5)
- moved Q3 10.2 mm to (27.3, 167.6)
- moved D6 10.1 mm to (29.7, 161.0)
- moved R10 9.09 mm to (29.8, 167.6)
- moved J11 8.39 mm to (22.6, 153.2)
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Connections:
- J6 pad 1: +BATT -> Net-(D9-Pad2)
- J6 pad 2: unconnected-(J6-Pad2) -> +BATT
- J7 pad 1: +BATT -> Net-(D7-Pad2)
- J7 pad 2: unconnected-(J7-Pad2) -> +BATT
- Q1 pad 1: PWM_KEROSTART -> PWM_KERO
- Q1 pad 2: Net-(D9-Pad2) -> GND
- Q1 pad 3: GND -> Net-(D7-Pad2)
- Q3 pad 1: PWM_KERO -> PWM_KEROSTART
- Q3 pad 2: Net-(D7-Pad2) -> GND
- Q3 pad 3: GND -> Net-(D9-Pad2)
- U5 pad 10: PPM_PWM_STARTER -> PPM_PWM_PUMP2
- U5 pad 14: PPM_PWM_PUMP2_3.3 -> PPM_STARTER_3.3
- U5 pad 15: PPM_PWM_PUMP2 -> PPM_PWM_STARTER
- U5 pad 9: PPM_STARTER_3.3 -> PPM_PWM_PUMP2_3.3
Routing:
- net CS: track 0.00 -> 56.7 mm, vias 0 -> 1
- net CLK: track 0.00 -> 48.3 mm, vias 0 -> 1
- net MISO: track 0.00 -> 44.7 mm, vias 0 -> 3
- net PWM_GLOW: track 3.01 -> 38.9 mm, vias 0 -> 1
- net PPM_GAZ: track 19.1 -> 0.18 mm, vias 1 -> 0
- net +3.3V: track 30.1 -> 46.3 mm, vias 0 -> 1
- net AUX_5V: track 28.8 -> 13.1 mm, vias 0 -> 1
- net PPM_GAZ_5V: track 29.6 -> 14.6 mm, vias 0 -> 1
- net GND: track 40.1 -> 28.6 mm
- net +BATT: track 95.1 -> 105.6 mm
- net Net-(J10-Pad1): track 0.00 -> 8.82 mm
- net RPM: track 0.00 -> 7.55 mm
- net VBAT_ADC: track 1.36 -> 7.94 mm
- net PPM_PWM_PUMP1: track 10.4 -> 16.1 mm
- net Net-(J10-Pad2): track 0.00 -> 5.15 mm
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Other:
- board size 73 x 55.4 mm -> 72.5 x 48.3 mm

Commit message: PCB
Parts:
- BT1: footprint Battery:Battery_Panasonic_CR2032-VS1N_Vertical_CircularHoles -> Battery:BatteryHolder_Keystone_1058_1x2032; moved to B.Cu
- moved BT1 50.8 mm to (69.3, 185.2)
- moved C1 19.7 mm to (34.4, 160.2), turned to -90 degrees
- moved U2 6.68 mm to (72.8, 165.3)
- moved U5 5.76 mm to (51.4, 162.7)
Connections:
- D1 pad 1: VBAT_ADC -> V_CPU
- D2 pad 1: VBAT_ADC -> V_CPU
- U1 pad 1: VBAT_ADC -> V_CPU
Routing:
- net V_CPU: track 0.00 -> 91.6 mm
- net VBAT_ADC: track 7.94 -> 85.0 mm, vias 0 -> 4
- net +3.3V: track 46.3 -> 120.2 mm, vias 1 -> 2
- net GLOW_CURRENT: track 0.90 -> 69.1 mm, vias 0 -> 2
- net RPM: track 7.55 -> 66.2 mm, vias 0 -> 1
- net Net-(BT1-Pad1): track 0.00 -> 45.4 mm, vias 0 -> 1
- net PPM_PWM_PUMP1_3.3: track 0.00 -> 43.4 mm, vias 0 -> 1
- net PPM_STARTER_3.3: track 0.00 -> 43.2 mm, vias 0 -> 3
- net PWM_GLOW_3.3: track 0.00 -> 41.8 mm, vias 0 -> 1
- net PPM_PWM_PUMP2_3.3: track 0.00 -> 41.0 mm, vias 0 -> 1
- net AUX: track 0.00 -> 40.8 mm, vias 0 -> 1
- net PPM_GAZ: track 0.18 -> 36.8 mm, vias 0 -> 1
- net TX2: track 5.49 -> 41.3 mm, vias 0 -> 2
- net PWM_KERO_3.3: track 0.00 -> 29.9 mm, vias 0 -> 1
- net PWM_KEROSTART: track 1.65 -> 31.1 mm, vias 0 -> 3
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
Commit message: pcb
Parts:
- added BOOT1: BOOT, Capacitor_SMD:C_0603_1608Metric, F.Cu at (59.5, 171.6)
- added C5: C, Capacitor_SMD:C_0603_1608Metric, F.Cu at (80.6, 191.6)
- added C6: C, Capacitor_SMD:C_0603_1608Metric, F.Cu at (80.6, 190.1)
- added C7: 1µF, Capacitor_SMD:C_0603_1608Metric, F.Cu at (38.2, 164.7)
- added D18: BZV55C3V3, Diode_SMD:D_MiniMELF, F.Cu at (39.8, 159.2)
- added D19: BZV55C3V3, Diode_SMD:D_MiniMELF, F.Cu at (43.4, 165.7)
- added J19: UART0, Connector_PinHeader_2.54mm:PinHeader_1x03_P2.54mm_Vertical, F.Cu at (80.6, 182.7)
- added R13: 10K, Resistor_SMD:R_0603_1608Metric, F.Cu at (58.0, 171.6)
- added R14: 10K, Resistor_SMD:R_0603_1608Metric, B.Cu at (56.7, 176.0)
- C1: value C -> 1µF
- C2: value C -> 10nF
- R3, R5, R6: value R -> 10K
- R4: value R -> 2.7K
- U1: value ESP32-DevKitC -> ESP32-WROOM-32D
- moved U2 7.02 mm to (66.1, 167.4)
- moved U1 5.06 mm to (68.2, 182.6)
- moved BT1 3.57 mm to (66.8, 182.6), turned to 25 degrees
- moved D8 2.29 mm to (77.4, 163.2)
- moved D12 2.28 mm to (80.9, 163.2)
- moved D5 2.27 mm to (73.9, 163.1)
- moved D16 2.01 mm to (48.8, 183.8)
- moved J15 1.68 mm to (44.0, 191.3)
- moved J18 1.68 mm to (46.6, 191.3)
- moved J4 1.68 mm to (41.5, 191.3)
- moved C1 1.55 mm to (36.0, 160.2)
- moved D14 1.02 mm to (45.3, 183.8)
Connections:
- R5 pad 1: GLOW_CURRENT -> V_CPU
- R5 pad 2: GND -> Net-(U1-Pad3)
- U1 pad 1: V_CPU -> GND
- U1 pad 10: PPM_GAZ -> PPM_PWM_PUMP2_3.3
- U1 pad 11: unconnected-(U1-Pad11) -> PPM_GAZ
- U1 pad 12: unconnected-(U1-Pad12) -> PWM_GLOW_3.3
- U1 pad 13: unconnected-(U1-Pad13) -> PWM_KEROSTART_3.3
- U1 pad 14: unconnected-(U1-Pad14) -> PWM_KERO_3.3
- U1 pad 15: unconnected-(U1-Pad15) -> GND
- U1 pad 2: unconnected-(U1-Pad2) -> V_CPU
- U1 pad 23: unconnected-(U1-Pad23) -> GLOW_CURRENT
- U1 pad 25: PWM_KERO_3.3 -> Net-(U1-Pad25)
- U1 pad 26: unconnected-(U1-Pad26) -> VBAT_ADC
- U1 pad 27: PWM_KEROSTART_3.3 -> Net-(U1-Pad27)
- U1 pad 3: VBAT_ADC -> Net-(U1-Pad3)
- U1 pad 34: unconnected-(U1-Pad34) -> Net-(U1-Pad34)
- U1 pad 35: unconnected-(U1-Pad35) -> Net-(U1-Pad35)
- U1 pad 39: (no net) -> GND
- U1 pad 4: GLOW_CURRENT -> unconnected-(U1-Pad4)
- U1 pad 5: PPM_PWM_PUMP1_3.3 -> unconnected-(U1-Pad5)
- U1 pad 6: PPM_PWM_PUMP2_3.3 -> unconnected-(U1-Pad6)
- U1 pad 7: PWM_GLOW_3.3 -> unconnected-(U1-Pad7)
- U1 pad 9: unconnected-(U1-Pad9) -> PPM_PWM_PUMP1_3.3
Routing:
- net Net-(U1-Pad3): track 0.00 -> 84.7 mm, vias 0 -> 2
- net +BATT: track 83.9 -> 124.3 mm
- net GLOW_CURRENT: track 69.1 -> 34.3 mm
- net V_CPU: track 91.6 -> 117.9 mm, vias 0 -> 1
- net Net-(U1-Pad35): track 0.00 -> 23.2 mm, vias 0 -> 1
- net Net-(U1-Pad34): track 0.00 -> 21.5 mm, vias 0 -> 1
- net CLK: track 55.6 -> 39.6 mm
- net Net-(D4-Pad1): track 44.0 -> 28.9 mm, vias 2 -> 1
- net PPM_PWM_PUMP1: track 21.3 -> 8.72 mm
- net Net-(J16-Pad1): track 40.3 -> 28.4 mm, vias 2 -> 0
- net PPM_PWM_PUMP2_3.3: track 41.0 -> 29.9 mm
- net Net-(D14-Pad1): track 36.9 -> 26.7 mm, vias 0 -> 1
- net PPM_GAZ: track 36.8 -> 26.7 mm
- net CS: track 61.4 -> 52.0 mm
- net PPM_PWM_PUMP1_3.3: track 43.4 -> 34.5 mm
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Other:
- board size 72.5 x 48.3 mm -> 70 x 48.3 mm

Commit message: PCB
Parts:
- removed BT1: Battery_Cell, Battery:BatteryHolder_Keystone_1058_1x2032
- removed C5, C6: C, Capacitor_SMD:C_0603_1608Metric
- removed D1, D2: D_Schottky, Diode_SMD:D_SMA
- added C8: 22µF, Capacitor_SMD:C_0603_1608Metric, F.Cu at (80.5, 190.0)
- added C9: 0.1µF, Capacitor_SMD:C_0603_1608Metric, F.Cu at (80.6, 191.5)
- D17: value BZV55C3V3 -> SMF5V0A; footprint Diode_SMD:D_MiniMELF -> Diode_SMD:D_SMF
- moved R6 0.45 mm to (39.9, 168.1), turned to 0 degrees
Connections:
- C3 pad 1: +3.3V -> V_CPU
- C4 pad 1: +3.3V -> V_CPU
- D17 pad 1: +3.3V -> V_CPU
- J11 pad 2: +3.3V -> V_CPU
- U1 pad 23: GLOW_CURRENT -> unconnected-(U1-Pad23)
- U1 pad 26: VBAT_ADC -> unconnected-(U1-Pad26)
- U1 pad 29: CLK -> CS
- U1 pad 30: unconnected-(U1-Pad30) -> CLK
- U1 pad 37: CS -> MOSI
- U1 pad 4: unconnected-(U1-Pad4) -> VBAT_ADC
- U1 pad 5: unconnected-(U1-Pad5) -> GLOW_CURRENT
- U2 pad 1: +3.3V -> V_CPU
- U3 pad 4: +3.3V -> V_CPU
- U4 pad 2: +3.3V -> V_CPU
- U5 pad 1: +3.3V -> V_CPU
Routing:
- net +3.3V: track 114.3 -> 0.00 mm
- net V_CPU: track 117.9 -> 179.7 mm, vias 1 -> 2
- net GLOW_CURRENT: track 34.3 -> 79.5 mm
- net Net-(BT1-Pad1): track 44.5 -> 0.00 mm, vias 1 -> 0
- net +BATT: track 124.3 -> 89.1 mm
- net Net-(C7-Pad1): track 84.7 -> 53.4 mm, vias 2 -> 0
- net CLK: track 39.6 -> 70.6 mm
- net PPM_PWM_PUMP2_3.3: track 29.9 -> 47.0 mm
- net Net-(J19-Pad1): track 23.2 -> 40.2 mm, vias 1 -> 0
- net Net-(J19-Pad2): track 21.5 -> 36.0 mm
- net CS: track 52.0 -> 37.5 mm
- net Net-(D16-Pad1): track 36.5 -> 24.7 mm, vias 1 -> 0
- net RPM: track 73.0 -> 63.1 mm
- net AUX: track 39.5 -> 29.5 mm
- net TX2: track 43.1 -> 35.7 mm
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
Commit message: PCB
Parts:
- added C10: 0.1µF, Capacitor_SMD:C_0603_1608Metric, B.Cu at (32.1, 154.7)
- added C11: 0.1µF, Capacitor_SMD:C_0603_1608Metric, B.Cu at (36.1, 151.5)
- added C5: 0.1µF, Capacitor_SMD:C_0603_1608Metric, B.Cu at (62.0, 162.3)
- added C6: 0.1µF, Capacitor_SMD:C_0603_1608Metric, B.Cu at (48.4, 157.2)
- added GND: Conn_01x01_Male, Connector_PinHeader_1.00mm:PinHeader_1x01_P1.00mm_Vertical, F.Cu at (65.3, 168.5)
- added TCK: Conn_01x01_Male, Connector_PinHeader_1.00mm:PinHeader_1x01_P1.00mm_Vertical, F.Cu at (72.6, 171.4)
- added TDI: Conn_01x01_Male, Connector_PinHeader_1.00mm:PinHeader_1x01_P1.00mm_Vertical, F.Cu at (48.4, 162.7)
- added TDO: Conn_01x01_Male, Connector_PinHeader_1.00mm:PinHeader_1x01_P1.00mm_Vertical, F.Cu at (63.6, 168.5)
- added TMS: Conn_01x01_Male, Connector_PinHeader_1.00mm:PinHeader_1x01_P1.00mm_Vertical, F.Cu at (59.3, 164.6)
- moved R4 0.39 mm to (23.8, 160.9)
- moved R3 0.39 mm to (20.8, 160.9)
- moved R6 0.13 mm to (39.9, 168.3)
Connections:
- U1 pad 16: unconnected-(U1-Pad16) -> TCK
- U1 pad 23: unconnected-(U1-Pad23) -> TDO
Routing:
- net GLOW_CURRENT: track 79.5 -> 93.7 mm
- net CLK: track 70.6 -> 78.2 mm
- net TDO: track 0.00 -> 4.92 mm
- net Net-(D4-Pad1): track 24.8 -> 26.6 mm
- net TCK: track 0.00 -> 1.37 mm
- net PWM_KERO_3.3: track 36.9 -> 38.1 mm
- net PWM_KEROSTART_3.3: track 33.8 -> 34.8 mm
- net Net-(J10-Pad1): track 7.99 -> 8.94 mm
- net V_CPU: track 179.7 -> 180.6 mm
- net GND: vias 703 -> 492
Other:
- board size 70 x 48.3 mm -> 71.3 x 48.3 mm
