File: Hardware/jf-ecu32/jf-ecu32.kicad_pcb (KiCad board)
At the start: 2 copper layers, 71.3 x 48.3 mm, 78 parts, among them J1 GAZ, J10 k, J11 RPM, J12 S.PORT, J13 PPM/PWM, J14 PUMP1, J15 PUMP1, J16 PPM/PWM, J17 PUMP2, J18 PUMP2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

Commit message: PCB
Parts:
- removed C4: 22µF, Capacitor_SMD:CP_Elec_5x3
- removed D17: SMF5V0A, Diode_SMD:D_SMF
- removed GND, TCK, TDI, TDO, TMS: Conn_01x01_Male, Connector_PinHeader_1.00mm:PinHeader_1x01_P1.00mm_Vertical
- added D1: SMF5V0A, Diode_SMD:D_SMF, B.Cu at (60.4, 152.0)
- added GND1: Conn_01x01_Male, Connector_PinHeader_1.00mm:PinHeader_1x01_P1.00mm_Vertical, F.Cu at (65.8, 168.4)
- added TCK1: Conn_01x01_Male, Connector_PinHeader_1.00mm:PinHeader_1x01_P1.00mm_Vertical, F.Cu at (72.6, 171.7)
- added TDI1: Conn_01x01_Male, Connector_PinHeader_1.00mm:PinHeader_1x01_P1.00mm_Vertical, F.Cu at (48.4, 162.7)
- added TDO1: Conn_01x01_Male, Connector_PinHeader_1.00mm:PinHeader_1x01_P1.00mm_Vertical, F.Cu at (64.0, 168.4)
- added TMS1: Conn_01x01_Male, Connector_PinHeader_1.00mm:PinHeader_1x01_P1.00mm_Vertical, F.Cu at (59.3, 164.5)
- added U6: AMS1117-5.0, Package_TO_SOT_SMD:SOT-223-3_TabPin2, B.Cu at (53.6, 154.2)
- C3: value 0.1µF -> 22µF
- C8: footprint Capacitor_SMD:C_0603_1608Metric -> Capacitor_SMD:CP_Elec_5x3
- moved C8 45.5 mm to (52.4, 154.2)
- moved C5 6.79 mm to (59.9, 155.8)
Connections:
- C5 pad 1: V_CPU -> +5V
- C8 pad 1: V_CPU -> +5V
- U4 pad 3: VDC -> +5V
- U5 pad 1: V_CPU -> +5V
Routing:
- net +5V: track 0.00 -> 44.8 mm, vias 0 -> 9
- net +BATT: track 88.8 -> 131.1 mm, vias 0 -> 1
- net VDC: track 11.7 -> 0.00 mm
- net V_CPU: track 180.6 -> 175.7 mm
- net VBAT_ADC: track 87.2 -> 83.9 mm
- net GND: vias 492 -> 471

Commit message: PCB
Parts:
- added Q7: AO3401A, Package_TO_SOT_SMD:SOT-23, B.Cu at (29.0, 176.5)
- J19: footprint Connector_PinHeader_2.54mm:PinHeader_1x03_P2.54mm_Vertical -> Connector_PinHeader_2.54mm:PinHeader_1x04_P2.54mm_Vertical
- moved C5 15.4 mm to (44.9, 159.5), turned to 180 degrees
- moved C6 14.1 mm to (61.7, 161.8)
- moved J19 1.25 mm to (81.5, 181.9)
Connections:
- C11 pad 1: V_CPU -> 3.3V
- C3 pad 1: V_CPU -> 3.3V
- C6 pad 1: V_CPU -> 3.3V
- C9 pad 1: V_CPU -> 3.3V
- J11 pad 2: V_CPU -> +5V
- J19 pad 1: Net-(J19-Pad1) -> 3.3V
- J19 pad 2: Net-(J19-Pad2) -> Net-(U1-Pad35)
- J19 pad 3: GND -> Net-(U1-Pad34)
- R13 pad 1: V_CPU -> 3.3V
- R14 pad 2: V_CPU -> 3.3V
- R5 pad 1: V_CPU -> 3.3V
- U1 pad 2: V_CPU -> 3.3V
- U1 pad 34: Net-(J19-Pad2) -> Net-(U1-Pad34)
- U1 pad 35: Net-(J19-Pad1) -> Net-(U1-Pad35)
- U2 pad 1: V_CPU -> 3.3V
- U3 pad 4: V_CPU -> 3.3V
- U4 pad 2: V_CPU -> 3.3V
Routing:
- net V_CPU: track 175.7 -> 0.00 mm, vias 2 -> 0
- net 3.3V: track 0.00 -> 141.4 mm, vias 0 -> 3
- net Net-(J19-Pad1): track 40.2 -> 0.00 mm
- net Net-(U1-Pad35): track 0.00 -> 38.2 mm
- net Net-(U1-Pad34): track 0.00 -> 36.4 mm, vias 0 -> 1
- net Net-(J19-Pad2): track 36.0 -> 0.00 mm, vias 1 -> 0
- net +5V: track 44.8 -> 61.8 mm
- net Net-(D3-Pad2): track 13.9 -> 17.3 mm
- net +BATT: track 131.1 -> 133.8 mm
- net CLK: track 78.2 -> 79.4 mm
- net Net-(D4-Pad1): track 26.6 -> 26.1 mm
- net PPM_PWM_PUMP1_3.3: track 35.5 -> 36.1 mm
- net GLOW_CURRENT: track 93.7 -> 93.2 mm
- net GND: vias 471 -> 445

Commit message: PCB
Parts:
- removed D11, D12, D14, D16, D4, D5, D6, D8: D_Schottky, Diode_SMD:D_SMA
- added R15: 10K, Resistor_SMD:R_0603_1608Metric, F.Cu at (62.0, 170.4)
- added R16: 10K, Resistor_SMD:R_0603_1608Metric, B.Cu at (77.7, 172.7)
- moved TCK1 7.90 mm to (65.5, 168.3)
- moved Q7 6.22 mm to (28.2, 182.6)
- moved R8 2.88 mm to (36.6, 193.2)
- moved J18 2.87 mm to (47.1, 188.5)
- moved J15 2.86 mm to (44.3, 188.5)
- moved J4 2.85 mm to (41.5, 188.5)
- moved R7 2.31 mm to (36.6, 186.2)
- moved R11 1.82 mm to (36.6, 172.4)
- moved R9 1.56 mm to (36.6, 179.4)
- moved GND1 1.40 mm to (67.2, 168.3)
- moved Q6 1.27 mm to (32.4, 193.3)
- moved J17 0.89 mm to (22.7, 192.0)
- moved J14 0.64 mm to (22.7, 186.1)
- moved Q5 0.64 mm to (32.4, 186.3)
- moved J9 0.39 mm to (22.7, 180.1)
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Connections:
- Q7 pad 1: unconnected-(Q7-Pad1) -> BRAKE
- U1 pad 24: unconnected-(U1-Pad24) -> Net-(U1-Pad24)
- U1 pad 26: unconnected-(U1-Pad26) -> BRAKE
Routing:
- net BRAKE: track 0.00 -> 71.5 mm, vias 0 -> 8
- net +BATT: track 133.8 -> 143.1 mm
- net Net-(J13-Pad1): track 21.5 -> 30.5 mm
- net RPM: track 63.1 -> 54.8 mm
- net TCK: track 1.37 -> 9.49 mm
- net CLK: track 79.4 -> 71.6 mm
- net Net-(J3-Pad1): track 16.0 -> 22.7 mm
- net Net-(J16-Pad1): track 27.4 -> 34.1 mm
- net GLOW_CURRENT: track 93.2 -> 86.6 mm
- net PPM_GAZ_5V: track 19.9 -> 15.1 mm
- net AUX_5V: track 19.8 -> 15.1 mm
- net 3.3V: track 141.4 -> 145.7 mm, vias 3 -> 4
- net Net-(J13-Pad3): track 24.5 -> 20.9 mm
- net TX2: track 35.7 -> 32.1 mm
- net Net-(J3-Pad3): track 26.1 -> 22.6 mm
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Other:
- board size 71.3 x 48.3 mm -> 71.4 x 46 mm

Commit message: SCH + PCB
Parts:
- moved D13 0.21 mm to (30.7, 185.4)
Changed lines of the file:
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@@
   )
   (footprint "Diode_SMD:D_SMA" (layer "B.Cu")
-    (at 30.52 185.42 180)
+    (at 30.734 185.42 180)
     (descr "Diode SMA (DO-214AC)")
     (tags "Diode SMA (DO-214AC)")
@@
   (segment (start 22.78 185.42) (end 23.415 186.055) (width 2) (layer "F.Cu") (net 37))
   (segment (start 23.415 186.055) (end 29.87 186.055) (width 2) (layer "F.Cu") (net 37))
-  (segment (start 27.885 186.055) (end 23.415 186.055) (width 2) (layer "B.Cu") (net 37))
-  (segment (start 28.52 185.42) (end 27.885 186.055) (width 2) (layer "B.Cu") (net 37))
+  (segment (start 28.099 186.055) (end 23.415 186.055) (width 2) (layer "B.Cu") (net 37))
+  (segment (start 28.734 185.42) (end 28.099 186.055) (width 2) (layer "B.Cu") (net 37))
   (segment (start 23.415 186.055) (end 22.78 185.42) (width 2) (layer "B.Cu") (net 37))
   (segment (start 42.418 151.003) (end 16.383 151.003) (width 0.5) (layer "F.Cu") (net 38))
