File: Hardware/jf-ecu32/_autosave-jf-ecu32.7.kicad_sch (KiCad schematic)
At the start: 89 parts, among them J1 GAZ, J10 k, J11 RPM, J12 S.PORT, J13 PPM/PWM, J14 PUMP1, J15 PUMP1, J16 PPM/PWM, J17 PUMP2, J18 PUMP2, J19 EN, J2 AUX, J20 Conn_01x06, J21 Conn_01x07, J3 PPM/PWM, J4 STARTER, J5 GLOW, J6 VANNE KEROSTART, J7 VANNE KERO, J8 BATTERY 2S/3S, J9 STARTER, Q1 AO3400A, Q2 QM6006D, Q3 AO3400A, Q4 QM6006D, Q5 QM6006D, Q6 QM6006D, Q7 AO3400A, Q8 AO3400A, U1 ESP32-WROOM-32D, U2 4050, U3 MAX31855KASA, U4 AMS1117-3.3, U5 4050, U6 AMS1117-5.0, U7 OPA340NA, U8 LM4040DBZ-2.5, U9 INA219AxDCN

Commit message: PCB + SRC
Parts:
- J20: footprint Connector_JST:JST_PH_B6B-PH-K_1x06_P2.00mm_Vertical -> (none)
Changed lines of the file:
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@@
       (effects (font (size 1.27 1.27)) (justify left))
     )
-    (property "Footprint" "Connector_JST:JST_PH_B6B-PH-K_1x06_P2.00mm_Vertical" (at 242.57 31.75 0)
+    (property "Footprint" "" (at 242.57 31.75 0)
       (effects (font (size 1.27 1.27)) hide)
     )
