File: Hardware/jf-ecu32/_autosave-jf-ecu32.7.kicad_sch (KiCad schematic)
At the start: 109 parts, among them J1 GAZ, J10 k, J11 RPM, J12 S.PORT, J13 PPM/PWM, J14 PUMP1, J15 PUMP1, J16 PPM/PWM, J17 PUMP2, J18 PUMP2, J19 EN, J2 AUX, J20 Conn_01x06, J21 Conn_01x07, J22 Micro_SD_Card_Det1, J23 Conn_01x04, J24 Conn_01x05, J3 PPM/PWM, J4 STARTER, J5 GLOW, J6 VANNE KEROSTART, J7 VANNE KERO, J8 BATTERY 2S/3S, J9 STARTER, Q1 A49T, Q2 A49T, Q3 A49T, Q4 LR8726, Q5 LR8726, Q6 LR8726, Q7 A49T, Q8 A49T, Q9 FDD6685, U1 ESP32-WROOM-32D, U10 BMP280, U2 4050, U3 MAX31855KASA, U4 AMS1117-3.3, U5 4050, U6 AMS1117-5.0, U7 OPA340NA, U8 LM4040DBZ-2.5, U9 INA219AxDCN

Commit message: PCB RPM Filter adjusted
Parts:
- R18: value 20K -> 10K
- R21: value 20K -> 30K
Changed lines of the file:
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@@
       (effects (font (size 1.27 1.27)))
     )
-    (property "Value" "20K" (at 273.05 111.76 90)
+    (property "Value" "30K" (at 273.05 111.76 90)
       (effects (font (size 1.27 1.27)))
     )
@@
       (effects (font (size 1.27 1.27)) (justify right))
     )
-    (property "Value" "20K" (at 289.56 140.9699 0)
-      (effects (font (size 1.27 1.27)) (justify right))
-    )
+    (property "Value" "10K" (at 289.56 140.9699 0)
+      (effects (font (size 1.27 1.27)) (justify right))
+    )
