File: Hardware/jf-ecu32/jf-ecu32.7.kicad_sch (KiCad schematic)
At the start: 89 parts, among them J1 GAZ, J10 k, J11 RPM, J12 S.PORT, J13 PPM/PWM, J14 PUMP1, J15 PUMP1, J16 PPM/PWM, J17 PUMP2, J18 PUMP2, J19 EN, J2 AUX, J20 Conn_01x06, J21 Conn_01x07, J3 PPM/PWM, J4 STARTER, J5 GLOW, J6 VANNE KEROSTART, J7 VANNE KERO, J8 BATTERY 2S/3S, J9 STARTER, Q1 AO3400A, Q2 QM6006D, Q3 AO3400A, Q4 QM6006D, Q5 QM6006D, Q6 QM6006D, Q7 AO3400A, Q8 AO3400A, U1 ESP32-WROOM-32D, U2 4050, U3 MAX31855KASA, U4 AMS1117-3.3, U5 4050, U6 AMS1117-5.0, U7 OPA340NA, U8 LM4040DBZ-2.5, U9 INA219AxDCN

Commit message: PCB
Parts:
- added R25: 100K, Resistor_SMD:R_0603_1608Metric, symbol Device:R
- J20: footprint Connector_JST:JST_PH_B6B-PH-K_1x06_P2.00mm_Vertical -> (none)
Connections:
- net BR_MOSFET: now also R25.1; no longer Q7.3 (D)
- new net: Q7.3 (D), R25.2
Other:
- moved on the sheet: Q7
Changed lines of the file:
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@@
 (kicad_sch (version 20230121) (generator eeschema)
   (paper "A3")
-  (junction (at 271.78 185.42) (diameter 0) (color 0 0 0 0)
-  )
   (junction (at 123.19 30.48) (diameter 0) (color 0 0 0 0)
   )
@@
   (junction (at 303.53 29.21) (diameter 0) (color 0 0 0 0)
   )
-  (junction (at 264.16 200.66) (diameter 0) (color 0 0 0 0)
-  )
   (junction (at 223.52 74.93) (diameter 0) (color 0 0 0 0)
   )
@@
   (junction (at 203.2 214.63) (diameter 0) (color 0 0 0 0)
   )
+  (junction (at 270.51 200.66) (diameter 0) (color 0 0 0 0)
+  )
   (junction (at 317.5 68.58) (diameter 0) (color 0 0 0 0)
   )
@@
   (junction (at 200.66 245.11) (diameter 0) (color 0 0 0 0)
   )
+  (junction (at 275.59 185.42) (diameter 0) (color 0 0 0 0)
+  )
   (junction (at 381 161.29) (diameter 0) (color 0 0 0 0)
   )
@@
   (junction (at 355.6 209.55) (diameter 0) (color 0 0 0 0)
   )
+  (junction (at 278.13 185.42) (diameter 0) (color 0 0 0 0)
+  )
   (junction (at 384.81 120.65) (diameter 0) (color 0 0 0 0)
   )
@@
     (stroke (width 0) (type default))
   )
+  (wire (pts (xy 257.81 200.66) (xy 270.51 200.66))
+    (stroke (width 0) (type default))
+  )
   (wire (pts (xy 378.46 111.76) (xy 374.65 111.76))
     (stroke (width 0) (type default))
@@
     (stroke (width 0) (type default))
   )
+  (wire (pts (xy 278.13 185.42) (xy 284.48 185.42))
+    (stroke (width 0) (type default))
+  )
   (wire (pts (xy 194.31 62.23) (xy 204.47 62.23))
     (stroke (width 0) (type default))
@@
     (stroke (width 0) (type default))
   )
+  (wire (pts (xy 275.59 185.42) (xy 278.13 185.42))
+    (stroke (width 0) (type default))
+  )
   (wire (pts (xy 132.08 59.69) (xy 163.83 59.69))
     (stroke (width 0) (type default))
@@
     (stroke (width 0) (type default))
   )
-  (wire (pts (xy 264.16 200.66) (xy 280.67 200.66))
-    (stroke (width 0) (type default))
-  )
   (wire (pts (xy 1.27 166.37) (xy 19.05 166.37))
     (stroke (width 0) (type default))
@@
     (stroke (width 0) (type default))
   )
+  (wire (pts (xy 278.13 194.31) (xy 278.13 198.12))
+    (stroke (width 0) (type default))
+  )
   (wire (pts (xy 302.26 168.91) (xy 304.8 168.91))
     (stroke (width 0) (type default))
@@
     (stroke (width 0) (type default))
   )
+  (wire (pts (xy 270.51 200.66) (xy 280.67 200.66))
+    (stroke (width 0) (type default))
+  )
   (wire (pts (xy 198.12 69.85) (xy 194.31 69.85))
     (stroke (width 0) (type default))
@@
     (stroke (width 0) (type default))
   )
+  (wire (pts (xy 275.59 177.8) (xy 275.59 185.42))
+    (stroke (width 0) (type default))
+  )
   (wire (pts (xy 299.72 199.39) (xy 299.72 201.93))
     (stroke (width 0) (type default))
@@
     (stroke (width 0) (type default))
   )
-  (wire (pts (xy 271.78 185.42) (xy 284.48 185.42))
-    (stroke (width 0) (type default))
-  )
   (wire (pts (xy 238.76 231.14) (xy 242.57 231.14))
     (stroke (width 0) (type default))
@@
     (stroke (width 0) (type default))
   )
+  (wire (pts (xy 278.13 208.28) (xy 278.13 212.09))
+    (stroke (width 0) (type default))
+  )
   (wire (pts (xy 384.81 120.65) (xy 384.81 121.92))
     (stroke (width 0) (type default))
@@
     (stroke (width 0) (type default))
   )
+  (wire (pts (xy 278.13 185.42) (xy 278.13 186.69))
+    (stroke (width 0) (type default))
+  )
   (wire (pts (xy 373.38 152.4) (xy 373.38 153.67))
     (stroke (width 0) (type default))
@@
     (stroke (width 0) (type default))
   )
-  (wire (pts (xy 257.81 185.42) (xy 271.78 185.42))
+  (wire (pts (xy 257.81 185.42) (xy 275.59 185.42))
     (stroke (width 0) (type default))
   )
@@
     (stroke (width 0) (type default))
   )
-  (wire (pts (xy 257.81 200.66) (xy 264.16 200.66))
-    (stroke (width 0) (type default))
-  )
   (wire (pts (xy 359.41 228.6) (xy 373.38 228.6))
     (stroke (width 0) (type default))
@@
     (stroke (width 0) (type default))
   )
-  (wire (pts (xy 264.16 190.5) (xy 264.16 200.66))
+  (wire (pts (xy 270.51 203.2) (xy 270.51 200.66))
     (stroke (width 0) (type default))
   )
@@
     )
   )
-  (global_label "BR_MOSFET" (shape input) (at 279.4 185.42 90) (fields_autoplaced)
-    (effects (font (size 1.27 1.27)) (justify left))
-    (property "Intersheetrefs" "${INTERSHEET_REFS}" (at 279.4 171.81 90)
-      (effects (font (size 1.27 1.27)) (justify left) hide)
+  (global_label "BR_MOSFET" (shape input) (at 275.59 177.8 180) (fields_autoplaced)
+    (effects (font (size 1.27 1.27)) (justify right))
+    (property "Intersheetrefs" "${INTERSHEET_REFS}" (at 261.9006 177.8 0)
+      (effects (font (size 1.27 1.27)) (justify right) hide)
     )
   )
@@
       (effects (font (size 1.27 1.27)) (justify left))
     )
-    (property "Footprint" "Connector_JST:JST_PH_B6B-PH-K_1x06_P2.00mm_Vertical" (at 242.57 31.75 0)
+    (property "Footprint" "" (at 242.57 31.75 0)
       (effects (font (size 1.27 1.27)) hide)
     )
@@
     )
   )
-  (symbol (lib_id "power:GND") (at 271.78 195.58 0) (unit 1)
+  (symbol (lib_id "power:GND") (at 278.13 212.09 0) (unit 1)
     (in_bom yes) (on_board yes) (dnp no) (fields_autoplaced)
-    (property "Reference" "#PWR01" (at 271.78 201.93 0)
+    (property "Reference" "#PWR01" (at 278.13 218.44 0)
       (effects (font (size 1.27 1.27)) hide)
     )
-    (property "Value" "GND" (at 271.78 200.66 0)
+    (property "Value" "GND" (at 278.13 217.17 0)
       (effects (font (size 1.27 1.27)))
     )
-    (property "Footprint" "" (at 271.78 195.58 0)
+    (property "Footprint" "" (at 278.13 212.09 0)
       (effects (font (size 1.27 1.27)) hide)
     )
-    (property "Datasheet" "" (at 271.78 195.58 0)
+    (property "Datasheet" "" (at 278.13 212.09 0)
       (effects (font (size 1.27 1.27)) hide)
     )
@@
     )
   )
+  (symbol (lib_id "Device:R") (at 278.13 190.5 0) (unit 1)
+    (in_bom yes) (on_board yes) (dnp no) (fields_autoplaced)
+    (property "Reference" "R25" (at 280.67 189.2299 0)
+      (effects (font (size 1.27 1.27)) (justify left))
+    )
+    (property "Value" "100K" (at 280.67 191.7699 0)
+      (effects (font (size 1.27 1.27)) (justify left))
+    )
+    (property "Footprint" "Resistor_SMD:R_0603_1608Metric" (at 276.352 190.5 90)
+      (effects (font (size 1.27 1.27)) hide)
+    )
+    (property "Datasheet" "~" (at 278.13 190.5 0)
+      (effects (font (size 1.27 1.27)) hide)
+    )
+    (pin "1")
+    (pin "2")
+    (instances
+      (project "jf-ecu32.7"
+        (path "/89131591-836b-4344-93b0-14d6b2e32546"
+          (reference "R25") (unit 1)
+        )
+      )
+    )
+  )
   (symbol (lib_id "power:+2V5") (at 248.92 115.57 0) (unit 1)
     (in_bom yes) (on_board yes) (dnp no) (fields_autoplaced)
@@
     )
   )
-  (symbol (lib_id "Transistor_FET:AO3400A") (at 269.24 190.5 0) (unit 1)
+  (symbol (lib_id "Transistor_FET:AO3400A") (at 275.59 203.2 0) (unit 1)
     (in_bom yes) (on_board yes) (dnp no) (fields_autoplaced)
-    (property "Reference" "Q7" (at 275.59 189.23 0)
+    (property "Reference" "Q7" (at 281.94 201.93 0)
       (effects (font (size 1.27 1.27)) (justify left))
     )
-    (property "Value" "AO3400A" (at 275.59 191.77 0)
+    (property "Value" "AO3400A" (at 281.94 204.47 0)
       (effects (font (size 1.27 1.27)) (justify left))
     )
-    (property "Footprint" "Package_TO_SOT_SMD:SOT-23" (at 274.32 192.405 0)
+    (property "Footprint" "Package_TO_SOT_SMD:SOT-23" (at 280.67 205.105 0)
       (effects (font (size 1.27 1.27) italic) (justify left) hide)
     )
-    (property "Datasheet" "http://www.aosmd.com/pdfs/datasheet/AO3400A.pdf" (at 269.24 190.5 0)
+    (property "Datasheet" "http://www.aosmd.com/pdfs/datasheet/AO3400A.pdf" (at 275.59 203.2 0)
       (effects (font (size 1.27 1.27)) (justify left) hide)
     )

Commit message: pcb
Parts:
- removed R25: 100K, Resistor_SMD:R_0603_1608Metric, symbol Device:R
Connections:
- net BR_MOSFET: now also Q7.3 (D)
Other:
- moved on the sheet: Q7
Changed lines of the file:
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@@
 (kicad_sch (version 20230121) (generator eeschema)
   (paper "A3")
+  (junction (at 271.78 185.42) (diameter 0) (color 0 0 0 0)
+  )
   (junction (at 123.19 30.48) (diameter 0) (color 0 0 0 0)
   )
@@
   (junction (at 303.53 29.21) (diameter 0) (color 0 0 0 0)
   )
+  (junction (at 264.16 200.66) (diameter 0) (color 0 0 0 0)
+  )
   (junction (at 223.52 74.93) (diameter 0) (color 0 0 0 0)
   )
@@
   (junction (at 203.2 214.63) (diameter 0) (color 0 0 0 0)
   )
-  (junction (at 270.51 200.66) (diameter 0) (color 0 0 0 0)
-  )
   (junction (at 317.5 68.58) (diameter 0) (color 0 0 0 0)
   )
@@
   (junction (at 200.66 245.11) (diameter 0) (color 0 0 0 0)
   )
-  (junction (at 275.59 185.42) (diameter 0) (color 0 0 0 0)
-  )
   (junction (at 381 161.29) (diameter 0) (color 0 0 0 0)
   )
@@
   (junction (at 355.6 209.55) (diameter 0) (color 0 0 0 0)
   )
-  (junction (at 278.13 185.42) (diameter 0) (color 0 0 0 0)
-  )
   (junction (at 384.81 120.65) (diameter 0) (color 0 0 0 0)
   )
@@
     (stroke (width 0) (type default))
   )
-  (wire (pts (xy 257.81 200.66) (xy 270.51 200.66))
-    (stroke (width 0) (type default))
-  )
   (wire (pts (xy 378.46 111.76) (xy 374.65 111.76))
     (stroke (width 0) (type default))
@@
     (stroke (width 0) (type default))
   )
-  (wire (pts (xy 278.13 185.42) (xy 284.48 185.42))
-    (stroke (width 0) (type default))
-  )
   (wire (pts (xy 194.31 62.23) (xy 204.47 62.23))
     (stroke (width 0) (type default))
@@
     (stroke (width 0) (type default))
   )
-  (wire (pts (xy 275.59 185.42) (xy 278.13 185.42))
-    (stroke (width 0) (type default))
-  )
   (wire (pts (xy 132.08 59.69) (xy 163.83 59.69))
     (stroke (width 0) (type default))
@@
     (stroke (width 0) (type default))
   )
+  (wire (pts (xy 264.16 200.66) (xy 280.67 200.66))
+    (stroke (width 0) (type default))
+  )
   (wire (pts (xy 1.27 166.37) (xy 19.05 166.37))
     (stroke (width 0) (type default))
@@
     (stroke (width 0) (type default))
   )
-  (wire (pts (xy 278.13 194.31) (xy 278.13 198.12))
-    (stroke (width 0) (type default))
-  )
   (wire (pts (xy 302.26 168.91) (xy 304.8 168.91))
     (stroke (width 0) (type default))
@@
     (stroke (width 0) (type default))
   )
-  (wire (pts (xy 270.51 200.66) (xy 280.67 200.66))
-    (stroke (width 0) (type default))
-  )
   (wire (pts (xy 198.12 69.85) (xy 194.31 69.85))
     (stroke (width 0) (type default))
@@
     (stroke (width 0) (type default))
   )
-  (wire (pts (xy 275.59 177.8) (xy 275.59 185.42))
-    (stroke (width 0) (type default))
-  )
   (wire (pts (xy 299.72 199.39) (xy 299.72 201.93))
     (stroke (width 0) (type default))
@@
     (stroke (width 0) (type default))
   )
+  (wire (pts (xy 271.78 185.42) (xy 284.48 185.42))
+    (stroke (width 0) (type default))
+  )
   (wire (pts (xy 238.76 231.14) (xy 242.57 231.14))
     (stroke (width 0) (type default))
@@
     (stroke (width 0) (type default))
   )
-  (wire (pts (xy 278.13 208.28) (xy 278.13 212.09))
-    (stroke (width 0) (type default))
-  )
   (wire (pts (xy 384.81 120.65) (xy 384.81 121.92))
     (stroke (width 0) (type default))
@@
     (stroke (width 0) (type default))
   )
-  (wire (pts (xy 278.13 185.42) (xy 278.13 186.69))
-    (stroke (width 0) (type default))
-  )
   (wire (pts (xy 373.38 152.4) (xy 373.38 153.67))
     (stroke (width 0) (type default))
@@
     (stroke (width 0) (type default))
   )
-  (wire (pts (xy 257.81 185.42) (xy 275.59 185.42))
+  (wire (pts (xy 257.81 185.42) (xy 271.78 185.42))
     (stroke (width 0) (type default))
   )
@@
     (stroke (width 0) (type default))
   )
+  (wire (pts (xy 257.81 200.66) (xy 264.16 200.66))
+    (stroke (width 0) (type default))
+  )
   (wire (pts (xy 359.41 228.6) (xy 373.38 228.6))
     (stroke (width 0) (type default))
@@
     (stroke (width 0) (type default))
   )
-  (wire (pts (xy 270.51 203.2) (xy 270.51 200.66))
+  (wire (pts (xy 264.16 190.5) (xy 264.16 200.66))
     (stroke (width 0) (type default))
   )
@@
     )
   )
-  (global_label "BR_MOSFET" (shape input) (at 275.59 177.8 180) (fields_autoplaced)
-    (effects (font (size 1.27 1.27)) (justify right))
-    (property "Intersheetrefs" "${INTERSHEET_REFS}" (at 261.9006 177.8 0)
-      (effects (font (size 1.27 1.27)) (justify right) hide)
+  (global_label "BR_MOSFET" (shape input) (at 279.4 185.42 90) (fields_autoplaced)
+    (effects (font (size 1.27 1.27)) (justify left))
+    (property "Intersheetrefs" "${INTERSHEET_REFS}" (at 279.4 171.81 90)
+      (effects (font (size 1.27 1.27)) (justify left) hide)
     )
   )
@@
     )
   )
-  (symbol (lib_id "power:GND") (at 278.13 212.09 0) (unit 1)
+  (symbol (lib_id "power:GND") (at 271.78 195.58 0) (unit 1)
     (in_bom yes) (on_board yes) (dnp no) (fields_autoplaced)
-    (property "Reference" "#PWR01" (at 278.13 218.44 0)
+    (property "Reference" "#PWR01" (at 271.78 201.93 0)
       (effects (font (size 1.27 1.27)) hide)
     )
-    (property "Value" "GND" (at 278.13 217.17 0)
+    (property "Value" "GND" (at 271.78 200.66 0)
       (effects (font (size 1.27 1.27)))
     )
-    (property "Footprint" "" (at 278.13 212.09 0)
+    (property "Footprint" "" (at 271.78 195.58 0)
       (effects (font (size 1.27 1.27)) hide)
     )
-    (property "Datasheet" "" (at 278.13 212.09 0)
+    (property "Datasheet" "" (at 271.78 195.58 0)
       (effects (font (size 1.27 1.27)) hide)
     )
@@
     )
   )
-  (symbol (lib_id "Device:R") (at 278.13 190.5 0) (unit 1)
-    (in_bom yes) (on_board yes) (dnp no) (fields_autoplaced)
-    (property "Reference" "R25" (at 280.67 189.2299 0)
-      (effects (font (size 1.27 1.27)) (justify left))
-    )
-    (property "Value" "100K" (at 280.67 191.7699 0)
-      (effects (font (size 1.27 1.27)) (justify left))
-    )
-    (property "Footprint" "Resistor_SMD:R_0603_1608Metric" (at 276.352 190.5 90)
-      (effects (font (size 1.27 1.27)) hide)
-    )
-    (property "Datasheet" "~" (at 278.13 190.5 0)
-      (effects (font (size 1.27 1.27)) hide)
-    )
-    (pin "1")
-    (pin "2")
-    (instances
-      (project "jf-ecu32.7"
-        (path "/89131591-836b-4344-93b0-14d6b2e32546"
-          (reference "R25") (unit 1)
-        )
-      )
-    )
-  )
   (symbol (lib_id "power:+2V5") (at 248.92 115.57 0) (unit 1)
     (in_bom yes) (on_board yes) (dnp no) (fields_autoplaced)
@@
     )
   )
-  (symbol (lib_id "Transistor_FET:AO3400A") (at 275.59 203.2 0) (unit 1)
+  (symbol (lib_id "Transistor_FET:AO3400A") (at 269.24 190.5 0) (unit 1)
     (in_bom yes) (on_board yes) (dnp no) (fields_autoplaced)
-    (property "Reference" "Q7" (at 281.94 201.93 0)
+    (property "Reference" "Q7" (at 275.59 189.23 0)
       (effects (font (size 1.27 1.27)) (justify left))
     )
-    (property "Value" "AO3400A" (at 281.94 204.47 0)
+    (property "Value" "AO3400A" (at 275.59 191.77 0)
       (effects (font (size 1.27 1.27)) (justify left))
     )
-    (property "Footprint" "Package_TO_SOT_SMD:SOT-23" (at 280.67 205.105 0)
+    (property "Footprint" "Package_TO_SOT_SMD:SOT-23" (at 274.32 192.405 0)
       (effects (font (size 1.27 1.27) italic) (justify left) hide)
     )
-    (property "Datasheet" "http://www.aosmd.com/pdfs/datasheet/AO3400A.pdf" (at 275.59 203.2 0)
+    (property "Datasheet" "http://www.aosmd.com/pdfs/datasheet/AO3400A.pdf" (at 269.24 190.5 0)
       (effects (font (size 1.27 1.27)) (justify left) hide)
     )
@@
   )
   (symbol (lib_id "4xxx:4050") (at 19.05 152.4 0) (unit 7)
-    (in_bom yes) (on_board yes) (dnp no) (fields_autoplaced)
+    (in_bom yes) (on_board yes) (dnp no)
     (property "Reference" "U5" (at 25.4 151.1299 0)
       (effects (font (size 1.27 1.27)) (justify left))
