File: Hardware/jf-ecu32/jf-ecu32.8.kicad_pcb (KiCad board)
At the start: 2 copper layers, 71.3 x 48 mm, 107 parts, among them J1 GAZ, J10 k, J11 RPM, J12 S.PORT, J13 PPM/PWM, J14 PUMP1, J15 PUMP1, J16 PPM/PWM, J17 PUMP2, J18 PUMP2, J19 EN, J2 AUX, J22 Micro_SD_Card_Det1, J23 Conn_01x04, J24 Conn_01x05, J3 PPM/PWM, J4 STARTER, J5 GLOW, J6 VANNE KEROSTART, J7 VANNE KERO, J8 BATTERY 2S/3S, J9 STARTER, Q1 A49T, Q2 A49T, Q3 A49T, Q4 LR8726, Q5 LR8726, Q6 LR8726, Q7 A49T, Q8 A49T, Q9 FDD6685, U1 ESP32-WROOM-32D, U10 BMP280, U2 4050, U3 MAX31855KASA, U4 AMS1117-3.3, U5 4050, U6 AMS1117-5.0, U7 OPA340NA, U8 LM4040DBZ-2.5, U9 INA219AxDCN

Commit message: Save
Parts:
- J22: footprint Connector_Card:J_SD_Card-micro_socket_A -> JF-ECU32 Library:J_SD_Card-micro_socket_A
- R17: value 20K -> 200K
- R18: value 20K -> 10K
- R21: value 20K -> 100K
Connections:
- U10 pad 2: unconnected-(U10-CSB-Pad2) -> 3.3V
- U10 pad 5: unconnected-(U10-SDO-Pad5) -> 3.3V
Routing:
- net 3.3V: track 215.0 -> 217.4 mm
