File: Hardware/jf-ecu32/easyeda/jf-ecu32.kicad_sch (KiCad schematic)
At the start: 69 parts, among them J1 GAZ, J10 k, J11 RPM, J12 S.PORT, J13 PPM/PWM, J14 PUMP1, J15 PUMP1, J16 PPM/PWM, J17 PUMP2, J18 PUMP2, J19 UART0, J2 AUX, J3 PPM/PWM, J4 STARTER, J5 GLOW, J6 VANNE KEROSTART, J7 VANNE KERO, J8 BATTERY 2S/3S, J9 STARTER, Q1 AO3400A, Q2 QM6006D, Q3 AO3400A, Q4 QM6006D, Q5 QM6006D, Q6 QM6006D, U1 ESP32-WROOM-32D, U2 4050, U3 MAX31855KASA, U4 AMS1117-3.3, U5 4050

Commit message: PCB
Parts:
- added BT1: Battery_Cell, Battery:BatteryHolder_Keystone_1058_1x2032, symbol Device:Battery_Cell
- added C5, C6: C, Capacitor_SMD:C_0603_1608Metric, symbol Device:C
- added C?: 0.1µF, Capacitor_SMD:CP_Elec_5x3, symbol Device:C
- added D1, D2: D_Schottky, Diode_SMD:D_SMA, symbol Device:D_Schottky
- added U?: BMP280, Package_LGA:Bosch_LGA-8_2x2.5mm_P0.65mm_ClockwisePinNumbering, symbol Sensor_Pressure:BMP280
- renumbered C8 to C?, C9 to C?, D17 to D?
Connections:
- net +3.3V: now also D1.2 (A); no longer C?.1, C?.1, R13.1, R14.2, R5.1, U1.2 (VDD)
- net CLK: now also U?.4 (SCK)
- net GND: now also BT1.2 (-), C5.2, C6.2, C?.2, U?.1 (GND), U?.7 (GND)
- net MISO: now also U?.5 (SDO)
- net MOSI: now also U?.3 (SDI)
- new net: BT1.1 (+), D2.2 (A)
- new net V_CPU: C5.1, C6.1, C?.1, C?.1, C?.1, D1.1 (K), D2.1 (K), R13.1, R14.2, R5.1, U1.2 (VDD), U?.6 (VDDIO), U?.8 (VDD)
