File: Hardware/RPM/rpm/rpm.kicad_pcb (KiCad board)
At the start: 2 copper layers, 11 parts, among them J1 Conn_01x03_Male, U1 LM358, U2 KMZ10A

Commit message: RPM
Connections:
- C2 pad 2: unconnected-(C2-Pad2) -> Net-(U2-Pad1)
- U1 pad 3: unconnected-(U1-Pad3) -> Net-(U1-Pad3)
- U2 pad 1: unconnected-(U2-Pad1) -> Net-(U2-Pad1)
- U2 pad 3: unconnected-(U2-Pad3) -> Net-(U1-Pad3)
Routing:
- net Net-(U1-Pad3): track 0.00 -> 8.14 mm
- net Net-(U2-Pad1): track 0.00 -> 5.65 mm
Changed lines of the file:
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@@
   (net 1 "GND")
   (net 2 "Net-(C2-Pad1)")
-  (net 3 "unconnected-(C2-Pad2)")
+  (net 3 "Net-(U2-Pad1)")
   (net 4 "Net-(C3-Pad1)")
   (net 5 "Sig")
@@
   (net 9 "Net-(R3-Pad1)")
   (net 10 "Net-(R5-Pad1)")
-  (net 11 "unconnected-(U1-Pad3)")
+  (net 11 "Net-(U1-Pad3)")
   (net 12 "unconnected-(U1-Pad5)")
-  (net 13 "unconnected-(U2-Pad1)")
-  (net 14 "unconnected-(U2-Pad3)")
   (footprint "Package_SO:SSOP-8_3.9x5.05mm_P1.27mm" (layer "F.Cu")
     (at 101.219 55.245)
@@
       (net 7 "Net-(R1-Pad2)") (pinfunction "-") (pintype "input"))
     (pad "3" smd roundrect (at -2.675 0.635) (size 1.55 0.6) (layers "F.Cu" "F.Paste" "F.Mask") (roundrect_rratio 0.25)
-      (net 11 "unconnected-(U1-Pad3)") (pinfunction "+") (pintype "input"))
+      (net 11 "Net-(U1-Pad3)") (pinfunction "+") (pintype "input"))
     (pad "4" smd roundrect (at -2.675 1.905) (size 1.55 0.6) (layers "F.Cu" "F.Paste" "F.Mask") (roundrect_rratio 0.25)
       (net 1 "GND") (pinfunction "V-") (pintype "power_in"))
@@
       (net 2 "Net-(C2-Pad1)") (pintype "passive"))
     (pad "2" smd roundrect (at 0.95 0 270) (size 1 1.45) (layers "F.Cu" "F.Paste" "F.Mask") (roundrect_rratio 0.25)
-      (net 3 "unconnected-(C2-Pad2)") (pintype "passive"))
+      (net 3 "Net-(U2-Pad1)") (pintype "passive"))
     (model "${KICAD6_3DMODEL_DIR}/Capacitor_SMD.3dshapes/C_0805_2012Metric.wrl"
       (offset (xyz 0 0 0))
@@
     (fp_line (start -0.525 -0.635) (end 1.05 -0.635) (layer "F.Fab") (width 0.1))
     (pad "1" thru_hole rect (at 0 0 90) (size 1 1) (drill 0.65) (layers *.Cu *.Mask)
-      (net 13 "unconnected-(U2-Pad1)") (pinfunction "+Vo") (pintype "output"))
+      (net 3 "Net-(U2-Pad1)") (pinfunction "+Vo") (pintype "output"))
     (pad "2" thru_hole oval (at 0 1.27 90) (size 1 1) (drill 0.65) (layers *.Cu *.Mask)
       (net 1 "GND") (pinfunction "Gnd") (pintype "power_in"))
     (pad "3" thru_hole oval (at 0 2.54 90) (size 1 1) (drill 0.65) (layers *.Cu *.Mask)
-      (net 14 "unconnected-(U2-Pad3)") (pinfunction "-Vo") (pintype "output"))
+      (net 11 "Net-(U1-Pad3)") (pinfunction "-Vo") (pintype "output"))
     (pad "4" thru_hole oval (at 0 3.81 90) (size 1 1) (drill 0.65) (layers *.Cu *.Mask)
       (net 10 "Net-(R5-Pad1)") (pinfunction "Vcc") (pintype "power_in"))
@@
   (segment (start 104.775 51.054) (end 98.176 57.653) (width 0.25) (layer "B.Cu") (net 1))
   (segment (start 94.107 55.165) (end 94.107 57.023) (width 0.25) (layer "F.Cu") (net 2))
+  (segment (start 96.134 58.923) (end 96.906 59.695) (width 0.25) (layer "F.Cu") (net 3))
+  (segment (start 94.107 58.923) (end 96.134 58.923) (width 0.25) (layer "F.Cu") (net 3))
+  (segment (start 96.906 59.695) (end 96.906 62.23) (width 0.25) (layer "F.Cu") (net 3))
   (segment (start 110.0695 55.621) (end 110.0695 58.039) (width 0.25) (layer "F.Cu") (net 4))
   (segment (start 115.443 51.689) (end 115.443 53.086) (width 0.25) (layer "F.Cu") (net 5))
@@
   (segment (start 107.2755 55.88) (end 107.6565 55.499) (width 0.25) (layer "F.Cu") (net 9))
   (segment (start 100.716 62.23) (end 102.9735 62.23) (width 0.25) (layer "F.Cu") (net 10))
+  (segment (start 100.076 61.6) (end 99.446 62.23) (width 0.25) (layer "F.Cu") (net 11))
+  (segment (start 98.544 55.88) (end 100.076 55.88) (width 0.25) (layer "F.Cu") (net 11))
+  (segment (start 100.076 55.88) (end 100.076 61.6) (width 0.25) (layer "F.Cu") (net 11))
 )
